Commit message: Delete the dead files and cut the historical narrative from the comments
Deleted, none of them reachable from run_campaign.sh or any world / slam /
navigation launch file:
  - rtabmap_3d_slam.launch.save
  - config/rtabmap/{icp_odom_params,slam_params}.yaml in the three packages,
    which nothing has ever loaded
  - waypoint_recorder.py x3, superseded by route_mine.yaml +
    generate_waypoints.py (and its CMakeLists entries)
  - plot_loop_closure.py; analyze_metrics.py draws that figure
  - the off-pipeline benches: suspension_sim.py, rocker_2d.py,
    yaw_calibration.py, run_yaw_calibration.sh, analiza_calibracion.py
The test/ benches and banco_seguidor*.py stay: they cover live code.

Comments: the change history, superseded diagnoses and dated A/B diaries are
gone; the reasoning that still applies stays, condensed.  sim_config.yaml
1218 -> 676 lines, ensamblajeurdf.xacro 1584 -> 1363, route_mine.yaml
266 -> 195, and the same in run_campaign.sh, trajectory_follower.py,
lcmine.world (byte-identical in the three packages, as the parity check
requires), the three rtabmap_3d_slam.launch, the three world launches, the two
spawned SDF models and ensamblajeurdf.gazebo.

Nothing but comments changed: every file was verified line-by-line against its
previous version with comments stripped, and the rocker-bogie URDF expands to
the same robot.  Two deliberate exceptions: run_campaign.sh --help now prints
lines 2-31 so the usage block is not cut off, and two lines of prose that had
leaked out of a comment in rtabmap_3d_slam.launch (where roslaunch was reading
them as element text) are back inside it.

README: the scripts tree matches the tidied package and names what each entry
point does, plus a line on the offline benches under robot_metrics/test/.

Co-Authored-By: Claude Opus 5 <noreply@anthropic.com>

File: src/rocker_bogie/urdf/ensamblajeurdf.xacro (robot description, xacro)
@@ -1,35 +1,27 @@
 <?xml version="1.0" ?>
 <robot name="ensamblajeurdf" xmlns:xacro="http://www.ros.org/wiki/xacro">
-<!-- Geometric differential: a real beam and two rods.  The gearbox
-     version (<joint type="gearbox">, arg "differential") was removed on
-     2026-09-13: it tipped the vehicle over on the spawn drop. -->
+<!-- Geometric differential: a real beam and two rods.  A gearbox joint
+     imposes the same relation but leaves the roll freedom unrestrained,
+     and it tipped the vehicle over on the spawn drop. -->
 <xacro:arg name="differential_linkage" default="false"/>
 <!-- ============ ORIENTACION DEL VARILLAJE DEL DIFERENCIAL ============
-     true  (defecto desde 2026-09-16): BARRAS LONGITUDINALES.  La viga rola
-           sobre el eje VERTICAL (Z) y sus dos extremos barren en +-x, asi
-           que las dos varillas van horizontales y a lo largo del vehiculo,
-           de la viga a un punto 53.192 mm POR DEBAJO del eje de cada rocker.
-     false: la de antes, TRANSVERSAL.  La viga rola sobre el eje de balanceo
-           (X), sus extremos suben y bajan, y las varillas bajan inclinadas
-           55 grados hasta el soporte de BarraBR, 50.9 mm por delante del eje
-           del rocker.  Es el varillaje con el que se midieron drop3 y drop4,
-           asi que para comparar con esas corridas hay que poner false.
-     LAS DOS DAN EL MISMO ACOPLAMIENTO, y esa es la cuenta que importa.  Con
-     la viga en Z, su extremo izquierdo avanza +y_off*sin(psi) y el derecho
-     -y_off*sin(psi): en OPOSICION.  Un punto del rocker a dz del eje avanza
-     dz*theta al cabecear.  Con una barra rigida a lo largo de x, el avance
-     del extremo de la viga y el del enganche son el mismo, asi que
+     true (defecto): BARRAS LONGITUDINALES.  La viga rola sobre el eje
+     VERTICAL (Z) y sus extremos barren en +-x, asi que las varillas van
+     horizontales y a lo largo del vehiculo, de la viga a un punto 53.192 mm
+     por debajo del eje de cada rocker.  false: TRANSVERSAL, la viga rola
+     sobre el eje de balanceo (X) y las varillas bajan inclinadas 55 grados.
+     LAS DOS DAN EL MISMO ACOPLAMIENTO.  Con la viga en Z, su extremo
+     izquierdo avanza +y_off*sin(psi) y el derecho -y_off*sin(psi), en
+     OPOSICION; un punto del rocker a dz del eje avanza dz*theta al cabecear,
+     y con barra rigida los dos avances son el mismo, asi que
          +y_off sin(psi) = dz*theta_izq      -y_off sin(psi) = dz*theta_der
      y sumando sale theta_izq + theta_der = 0, que es el diferencial.
-     POR QUE NO VALE SOLO CAMBIAR EL <axis> A Z dejando lo demas: con la viga
-     transversal y las varillas colgando, girar en Z mueve los enganches
-     23.2 mm en X y 0.0 en Z (a 10 grados), o sea las varillas no suben ni
-     bajan y el diferencial deja de acoplar.  Medido antes de tocar nada.
-     LO QUE CUESTA: la viga baja de z 0.673472 a 0.523472 en el marco del
-     chasis, o sea de asomar 38 mm por encima del techo a quedarse DENTRO de
-     la caja del chasis, y las varillas pasan a correr por la panza, 8.5 mm
-     por encima de ella.  Ninguno de los tres eslabones lleva colision, asi
-     que la fisica no simula esa interferencia; en un vehiculo de verdad hay
-     que dejarles el hueco.
+     NO BASTA CON CAMBIAR EL <axis> A Z: con la viga transversal y las
+     varillas colgando, girar en Z mueve los enganches 23.2 mm en X y 0.0 en Z
+     (a 10 grados), o sea las varillas no suben ni bajan y deja de acoplar.
+     LO QUE CUESTA: la viga queda DENTRO de la caja del chasis y las varillas
+     corren por la panza, 8.5 mm por encima.  Ninguno de los tres eslabones
+     lleva colision, asi que la fisica no simula esa interferencia; en un
+     vehiculo de verdad hay que dejarles el hueco.
      =================================================================== -->
 <xacro:arg name="diff_longitudinal" default="true"/>
@@ -43,115 +35,59 @@
                          '$(arg differential_linkage)' == 'true'}"/>
 <!-- TOPE SUPERIOR DE LOS BOGIES (rev_3 / rev_4), en radianes.
-     SUBIDO DE 0.6 A 1.0 EL 2026-09-10, y es una hipotesis a contrastar, no un
-     valor asentado.  Medido sobre metrics_rocker_bogie_diagnostic/run01, una
-     vuelta de 135.8 m con los pivotes ya registrados:
-                        recorrido usado        toca +0.6   toca -0.6
-       rockers          -8.9 .. +8.2 deg  25%      0.00 %     0.00 %
-       rev_3 (bogie)   -19.0 .. +34.4 deg 100%     1.88 %     0.00 %
-       rev_4 (bogie)   -25.9 .. +34.4 deg 100%     0.06 %     0.00 %
-     Los dos pivotes llevaban el mismo +-0.6 rad: al rocker le sobran tres
-     cuartos y al bogie le falta, y le falta SOLO por arriba.  Y saturar no es
-     inocuo: con el bogie en el tope hay rueda en el aire el 100 % del tiempo,
-     sin una sola excepcion en la corrida; con las seis apoyadas, el tope no se
-     toca nunca (0.00 %).  La descarga previa al despegue es gradual (fuerza
-     normal 1.00 -> 0.12 en 200 ms), o sea el mecanismo se queda sin geometria,
-     no es un rebote de contacto.
-     PROBADO 1.0 Y ES PEOR.  MUCHO PEOR.  No ampliar sin leer esto.
-     A/B a igual seed, ruta y LiDAR, sobre el tramo que las dos corridas
-     recorrieron (0 - 52.2 m):
+     NO AMPLIAR SIN LEER ESTO.  Sobre una vuelta completa los bogies usan todo
+     su recorrido y tocan el tope superior, asi que parece que 0.6 ata.  El
+     A/B a igual seed, ruta y LiDAR dice lo contrario:
                               0.6        1.0
        n<6                   21.5 %     64.6 %
        n<=4                   8.1 %     40.5 %
-       contacto Rueda_3_1    91.5 %     39.8 %
-       contacto Rueda_1_1    96.7 %     62.0 %
        rev_4 en su tope       0.16 %    49.52 %
        final                 135.8 m    VUELCO en 54.2 m (roll -112 deg)
-     Y el detalle que lo explica: con 1.0, rev_4 se enrolla hasta +57.3 deg en
-     el metro 17.7 y SE QUEDA CLAVADO AHI 25 metros seguidos.  Durante los
-     metros 20-40 la Rueda_3_1 esta en el aire el 100 % del tiempo y el
-     vehiculo rueda sobre cuatro.  Ese tramo es el LLANO, donde la corrida de
-     0.6 pierde contacto el 3.2 % y el 0.0 %.  No es el terreno pidiendo mas
-     recorrido: el balancin se va a tope y se aparca.
-     O SEA: el +-0.6 no ataba, SOSTENIA.  El tope estaba cargando el vehiculo.
-     Es el mismo sintoma que rocker_pivot_zero_note (sim_config.yaml) apunto en
-     los rockers -"pivots are DRIVEN to whatever stop exists", 34 deg -> 56 deg
-     al ampliar- y que quedo como "causa no encontrada".  Ahora se sabe que no
-     es especifico de los rockers: le pasa igual a los bogies, y el sentido es
-     siempre el mismo (+, nunca -).
-     HIPOTESIS PARA LA PROXIMA, no comprobada: el par de reaccion del motor de
-     la rueda.  Las ruedas van con controlador de velocidad y la reaccion cae
-     sobre el eslabon que lleva la articulacion, o sea el propio balancin.  Sin
-     nada que la equilibre -no hay muelle, y damping/friction solo resisten, no
-     devuelven- un par constante enrolla el pivote hasta donde le dejen.  Se
-     contrasta mirando si el enrollamiento sigue al par de rueda y si afloja al
-     parar o al retroceder: en el metro 45-50 rev_4 si aflojo (+5.1 deg) y la
-     Rueda_3_1 recupero el 55 % de contacto.
-     Mientras eso no se resuelva, ampliar el tope solo mueve el problema mas
-     lejos.  Se queda en 0.6, que es donde estaba.
-     EL LOWER NO SE TOCA a proposito: se queda en -0.6 y el maximo medido es
-     -25.9 deg, asi que no ata.  Cambiar solo lo que la hipotesis dice.
-     OJO, NO REPETIR EL FALLO DE LOS ROCKERS: ampliar +-0.6 a +-1.0 en
-     rocker_pivot_* empeoro las cosas y quedo como "causa no encontrada" en
-     rocker_pivot_zero_note (sim_config.yaml).  Ahora se sabe por que: se le dio
-     recorrido al pivote que iba sobrado.  Los rockers siguieron en +-0.6
-     hasta el 2026-09-13, cuando se ampliaron a +-1.0 a peticion: con el
-     varillaje del diferencial usan como mucho ~7 deg y no tocan el tope,
-     asi que el aviso de arriba ya no aplica a ellos (a los bogies SI).
-     A/B: differential_linkage y lo demas igual, y bogie_upper:=0.6 reproduce
-     el modelo con el que se tomo la corrida de referencia. -->
+     Con 1.0, rev_4 se enrolla hasta +57.3 deg en el metro 17.7 y SE QUEDA
+     CLAVADO AHI 25 metros -en el LLANO- con la Rueda_3_1 en el aire el 100 %
+     del tiempo.  El tope no ataba: SOSTENIA.
+     HIPOTESIS, no comprobada: el par de reaccion del motor de la rueda.  Las
+     ruedas van con controlador de velocidad y la reaccion cae sobre el propio
+     balancin; sin nada que la equilibre -no hay muelle, y damping/friction
+     solo resisten, no devuelven- un par constante enrolla el pivote hasta
+     donde le dejen.  Mientras eso no se resuelva, ampliar el tope solo mueve
+     el problema mas lejos.
+     EL LOWER NO SE TOCA: el maximo medido es -25.9 deg, asi que no ata.  Los
+     rockers SI llevan +-1.0: con el varillaje del diferencial usan como mucho
+     ~7 deg y no tocan el tope.  El aviso de arriba es de los BOGIES. -->
 <xacro:arg name="bogie_upper" default="0.6"/>
 <!-- ALTURA DEL PIVOTE DEL BOGIE (rev_3 / rev_4): cuanto se BAJA, en metros.
-     0.0 = el modelo de siempre, byte a byte.  El pivote esta hoy 0.529 m sobre
-     la huella de contacto (0.351 sobre el eje, mas el radio 0.178).
      POR QUE ES UNA PALANCA.  El par de una rueda llega al brazo por DOS
      caminos que suman: la reaccion -e en el eje, y la fuerza de traccion e/r
-     aplicada en la huella, que cuelga de ese brazo de 0.529 m.  El total es
+     aplicada en la huella, que cuelga del brazo del pivote.  El total es
          M_motor = K * ( -(e_media + e_trasera) ),   K = h_huella / r
-     con K = 0.529/0.178 = 2.97 hoy.  Medido sobre
-     metrics_rocker_bogie_par_ruedas/run01 (135.5 m): K ajustado 3.15 (rev_4,
-     r=-0.93) y 3.07 (rev_3, r=-0.96), y el balance estatico del pivote cierra
-     con residuo -0.05 y -0.78 N*m.  M_motor positivo levanta la rueda MEDIA,
-     que es justo la peor de las seis en contacto (94.2 % y 92.2 %).
-     Despega con M_motor ~ +50 N*m = 8.4 N*m por rueda, menos de la mitad del
-     limite de 20.
-     K escala LINEAL con esta altura: K = (0.529 - bogie_drop) / 0.178.
-       0.100 -> K 2.41 (-19 %)
-       0.178 -> K 1.97 (-34 %)
-       0.351 -> K 1.00 (-66 %), el pivote a la altura del EJE
-     1.00 es el suelo: ahi ya solo queda la reaccion en el eje, porque la
-     huella siempre esta un radio por debajo.
+     Ajustado sobre una corrida de 135.5 m: K 3.15 (rev_4, r=-0.93) y 3.07
+     (rev_3, r=-0.96), con el balance estatico del pivote cerrando con residuo
+     -0.05 y -0.78 N*m.  M_motor positivo levanta la rueda MEDIA, que es la
+     peor de las seis en contacto, y despega con ~8.4 N*m por rueda, menos de
+     la mitad del limite de 20.  K escala LINEAL con esta altura,
+     K = (0.529 - bogie_drop) / 0.178, y su suelo es 1.00: ahi solo queda la
+     reaccion en el eje, porque la huella siempre esta un radio por debajo.
      QUE MUEVE Y QUE NO.  Solo baja el EJE del pivote y el soporte que cuelga
      de el (Acople_Rodamiento_*_1: 1.4 kg, visual e inercia, sin colision).
      Los cuatro hijos (link_r_15..18) se suben lo mismo, asi que las seis
-     ruedas, los brazos del balancin (-0.189 media / +0.237 trasera) y la
-     altura de reposo quedan EXACTAMENTE donde estaban -> spawn_z no se toca.
-     Lo comprueba src/robot_metrics/test/test_bogie_drop.py, que es el fallo
-     silencioso: bajar el pivote sin compensar hunde media suspension.
-     LA HUELLA DE APOYO NO SE PAGA, SE GANA.  En reposo es identica: 0.5383 m2,
-     batalla 0.8532, via 0.6775, las seis ruedas coplanarias.  Deflectado si
-     cambia, y a favor: hoy el brazo pivote->rueda esta INCLINADO (dx -0.189,
-     dz -0.351), asi que girar el balancin echa la rueda hacia ATRAS ademas de
-     subirla: en el tope de +34.4 deg la rueda media retrocede 0.165 m, la
-     batalla se hunde a 0.613 y el area cae un 27 %, hasta 0.391 m2.  Con el
-     pivote a la altura del eje el brazo queda horizontal, la rueda apenas se
-     mueve en x (+0.033) y el area solo pierde un 6 %.  Con los angulos
-     medidos en metrics_rocker_bogie_par_ruedas/run01: area p05 0.480 ->
-     0.528 m2, y en el peor instante 0.391 -> 0.507 (+30 %).
-     Y EL RECORRIDO DE LA SUSPENSION NO SE TOCA.  El desnivel que traga el
-     balancin (rueda media contra trasera) es +0.241 m a 34.4 deg con drop 0
-     y con drop 0.351: depende solo de los brazos HORIZONTALES, que no se
-     mueven.  El tope de +-0.6 rad sigue valiendo para el mismo escalon.
+     ruedas, los brazos del balancin y la altura de reposo quedan EXACTAMENTE
+     donde estaban -> spawn_z no se toca.  Lo comprueba
+     src/robot_metrics/test/test_bogie_drop.py, porque el fallo es silencioso:
+     bajar el pivote sin compensar hunde media suspension.
+     LA HUELLA NO SE PAGA, SE GANA.  En reposo es identica.  Deflectada
+     cambia a favor: con el brazo pivote->rueda INCLINADO, girar el balancin
+     echa la rueda hacia atras ademas de subirla y el area cae un 27 % en el
+     tope; con el pivote a la altura del eje el brazo queda horizontal y solo
+     pierde un 6 %.  El recorrido de la suspension no se toca: el desnivel que
+     traga el balancin depende solo de los brazos HORIZONTALES.
      Como el varillaje, va por las DOS rutas de spawn del launch. -->
-<!-- TOPE DE bogie_drop, Y SE LO COME rocker_drop.  La cuenta de arriba
-     -0.178 -> K 1.97, 0.351 -> K 1.00- vale con rocker_drop = 0, que es cuando
-     el pivote del bogie sale de 0.351444 m sobre el eje.  Con rocker_drop en su
-     defecto (0.343839) el montante comun ya lo ha bajado a 0.178, o sea
+<!-- TOPE DE bogie_drop, Y SE LO COME rocker_drop.  La cuenta de arriba vale
+     con rocker_drop = 0; con el montante comun ya bajado,
          tope de bogie_drop = 0.351444 - max(0, rocker_drop - 0.170395)
-     y con el defecto eso son 0.178 m EXACTOS, no 0.351.  Pasarse no da error:
-     mete el eje del bogie POR DEBAJO del plano de las ruedas, con lo que la
-     huella deja de estar un radio por debajo del pivote y K vuelve a subir por
-     el otro lado.  Las dos palancas ya estan igualadas en K = 2.00 con
-     bogie_drop = 0, asi que este arg solo hace falta para desnivelarlas a
-     proposito.  Lo comprueba test_bogie_drop.py (seccion 2). -->
+     Pasarse no da error: mete el eje del bogie POR DEBAJO del plano de las
+     ruedas, con lo que la huella deja de estar un radio por debajo del pivote
+     y K vuelve a subir por el otro lado.  Con el defecto las dos palancas ya
+     estan igualadas con bogie_drop = 0, asi que este arg solo hace falta para
+     desnivelarlas a proposito.  Lo comprueba test_bogie_drop.py (seccion 2). -->
 <xacro:arg name="bogie_drop" default="0.0"/>
 <xacro:property name="bogie_drop" value="$(arg bogie_drop)"/>
@@ -163,79 +99,47 @@
      toca: misma altura, misma guarda al suelo, misma altura de sensores.
      POR QUE.  La huella de apoyo era 0.5383 m2 contra 0.3996 del tracked y
-     0.2923 del husky.  Con 0.862 queda en 0.4000 m2, la del tracked al 0.1 %.
-     Batalla 0.8532 -> 0.7355, via 0.7821 -> 0.5840.
+     0.2923 del husky; con 0.862 queda en 0.4000 m2, la del tracked al 0.1 %.
      0.862 ES EL MINIMO: las ruedas quedan a 0.3677 m entre centros, 11.7 mm
-     de holgura entre llantas de 0.178 m.  Menos factor y chocan, y encoger la
-     rueda rompe el radio igualado de las tres plataformas.
+     de holgura entre llantas, y encoger la rueda rompe el radio igualado de
+     las tres plataformas.
      Se escalan solo los origin de los joint y las pose de los joints de bola;
      NO los origin de dentro de los link: las piezas no cambian de tamaño,
-     solo se acercan, asi que conservan masa e inercia.  Las mallas no
-     encogen, asi que los eslabones estructurales se solapan un poco en
-     pantalla; ninguno tiene colision salvo las seis ruedas.
-     bogie_drop sube a 0.227 (K 1.70) porque el margen contra el despegue
-     escala con el brazo del balancin, que pasa a -0.1632 / +0.2046.
-     MEDIDO con esta geometria (metrics_rocker_bogie_drop3): n<6 = 11.37 %,
-     contra 4.91 % con la huella grande y el mismo K.  Encoger la huella
-     CUESTA contacto, sobre todo en las delanteras (96.51 / 95.01).
+     solo se acercan, asi que conservan masa e inercia.
+     CUESTA CONTACTO: con esta geometria n<6 = 11.37 % contra 4.91 % con la
+     huella grande y el mismo K, sobre todo en las delanteras.
      ========================================================== -->
 <!-- ==================== ALTURA DEL ROCKER ====================
      rocker_drop: cuanto se ACORTA, en metros, la caida vertical del brazo del
-     rocker entre su pivote y el eje de las ruedas.  0.0 = el modelo de CAD.
-     QUE ERA.  El pivote del rocker estaba 0.5219 m por encima del plano de
-     los ejes, o sea 0.6999 m sobre la huella de contacto, con lo que
-         K_rocker = h_huella / r = 0.6999 / 0.178 = 3.93
-     contra 2.98 del bogie con bogie_drop = 0.  Es la misma palanca que la
-     nota de bogie_drop describe, y la del rocker era la mayor de las dos.  El
-     chasis quedaba 0.638 m sobre el suelo con las ruedas de 0.178: una mesa
-     sobre zancos, no un rover.
+     rocker entre su pivote y el eje de las ruedas.  0.0 = el modelo de CAD,
+     que dejaba el pivote 0.6999 m sobre la huella -K_rocker = 3.93 contra
+     2.98 del bogie- y el chasis 0.638 m sobre el suelo: una mesa sobre
+     zancos, no un rover.
      QUE HACE.  Acorta las DOS ramas del rocker en la misma cantidad, asi que
      las seis ruedas suben lo mismo y siguen coplanarias:
-       * rama delantera - link_r_21 / link_r_22 (BarraBR -> ApoyoServomotor),
-         -0.256945 m de caida, se le resta rocker_drop entero.
-       * rama trasera   - link_r_7/8, link_r_9/10, link_r_11/12, 0.170395 m
-         de caida en total, se escalan las tres por rk_rear para que la rama
-         siga bajando de forma monotona en vez de doblarse.
-     LO QUE NO TOCA: nada en x ni en y.  Batalla, via, area de apoyo, brazos
-     del balancin y los tres parametros de twist_to_wheels se quedan
-     exactamente donde estaban.  Tampoco toca bogie_drop: el pivote del bogie
-     conserva su altura RELATIVA al brazo, asi que las dos palancas se pueden
-     mover por separado.  Tampoco toca link_r_5 / link_r_6, que es donde el
-     varillaje del diferencial cierra sus ball joints (-0.053192): el enganche
-     sigue siendo valido sin recalcular el varillaje.
-     SALE DE DOS SITIOS, Y EL PRIMERO SE AGOTA EN 0.170395 m.
-     TRAMO 1, hasta 0.170395: lo paga la RAMA TRASERA del rocker, que se va
-     aplanando.  0.170395 es exactamente lo que el pivote del rocker estaba por
-     encima del del bogie (0.5219 contra 0.3515 sobre los ejes), asi que al
-     agotarlo los DOS PIVOTES QUEDAN A LA MISMA ALTURA y la rama trasera queda
-     horizontal: el dibujo de libro del mecanismo.  Ahi K_rocker pasa de 3.93 a
-     2.97, la del bogie con bogie_drop = 0.  Mas alla, rk_rear seria negativo y
-     la rama subiria antes de bajar, asi que el tramo se cierra.
-     TRAMO 2, otros 0.211702: lo paga el MONTANTE COMUN, lo que hay entre el
-     extremo de cada brazo y el eje de su rueda.  Las SEIS ruedas lo comparten,
-     asi que encogerlo baja los dos pivotes A LA VEZ y en la misma cantidad:
-     siguen nivelados y los brazos no cambian de forma.  Por eso la ESTRUCTURA
-     SE CONSERVA: lo unico que encoge es el montaje de la rueda.
-     Y SE GASTA EN DOS PARTES, PORQUE NO SON LO MISMO.  El montante tiene
-     encima la junta de direccion (rev_5..8 en las cuatro ruedas de las
-     esquinas) y debajo la MANGUETA, que es la pieza que gira con ella:
+       * rama delantera - link_r_21 / link_r_22, -0.256945 m de caida, se le
+         resta rocker_drop entero.
+       * rama trasera   - link_r_7/8, 9/10, 11/12, 0.170395 m en total, se
+         escalan por rk_rear para que la rama siga bajando de forma monotona.
+     LO QUE NO TOCA: nada en x ni en y -batalla, via, area de apoyo, brazos
+     del balancin y los tres parametros de twist_to_wheels se quedan donde
+     estaban-, ni bogie_drop, ni link_r_5 / link_r_6, que es donde el varillaje
+     del diferencial cierra sus ball joints.
+     SALE DE DOS SITIOS.  TRAMO 1, hasta 0.170395: lo paga la RAMA TRASERA,
+     que se va aplanando; 0.170395 es exactamente lo que el pivote del rocker
+     estaba por encima del del bogie, asi que al agotarlo LOS DOS PIVOTES
+     QUEDAN A LA MISMA ALTURA (K_rocker 3.93 -> 2.97) y la rama trasera queda
+     horizontal.  Mas alla rk_rear seria negativo y la rama subiria antes de
+     bajar.  TRAMO 2, otros 0.211702: lo paga el MONTANTE COMUN, que comparten
+     las SEIS ruedas, asi que baja los dos pivotes a la vez y en la misma
+     cantidad: la ESTRUCTURA SE CONSERVA y lo unico que encoge es el montaje
+     de la rueda.  Y se gasta en dos partes porque no son lo mismo:
        2a. rev_5..8 y link_r_25/26, 0.074002 m: del extremo del brazo a la
-           junta de direccion.  Esto SI se gasta entero primero; al agotarlo la
-           junta queda en el propio extremo del brazo, que es donde va.
-       2b. link_r_27..32, 0.137700 m: la MANGUETA, el poste VERTICAL que cuelga
-           de la junta de direccion y del que cuelga la rueda.  Es el eje de
-           giro de la direccion en persona, asi que dejarlo sin altura hace que
-           las ruedas de las esquinas giren sobre un muñon de milimetros.  Se
-           gasta el ULTIMO y el defecto le deja el 60 %.
-     REPARTO NUEVO 2026-09-13: link_r_33..38 (soporte del motor) pasa de
-     "0 +-0.0270927 -0.05865" a "0 +-0.0270927 0", o sea a ser un brazo
-     PURAMENTE HORIZONTAL, y sus 0.05865 m de caida se los queda link_r_27..32.
-     El total no cambia -las ruedas siguen donde estaban- pero la union pasa a
-     leerse como lo que es: poste vertical a 90 grados + salida lateral al eje.
-     Antes la caida iba repartida entre los dos y la mangueta salia en diagonal.
+           junta de direccion.  Se gasta entero primero.
+       2b. link_r_27..32, 0.137700 m: la MANGUETA, el poste VERTICAL del que
+           cuelga la rueda y que ES el eje de giro de la direccion.  Se gasta
+           el ULTIMO y el defecto le deja el 60 %.
      TECHO 0.382097 = 0.170395 + 0.074002 + 0.137700.  Ahi la mangueta es cero
-     y la rueda colgaria del brazo. No llegar.
-     0.299477 POR DEFECTO, que deja la mangueta en el 60 % (82.6 mm).  Se
-     probo 0.239200 (K 2.59, mangueta entera) el 2026-09-13 y se volvio aqui
-     el mismo dia.  Con 0.299477:
+     y la rueda colgaria del brazo.  No llegar.
+     0.299477 POR DEFECTO:
          pivote del rocker  0.5219 -> 0.2224 m sobre los ejes
          K_rocker             3.93 -> 2.25
@@ -243,19 +147,15 @@
          panza del chasis    0.638 -> 0.338 m sobre el suelo
      EL COMPROMISO ES EXPLICITO: la mangueta y K tiran en contra.  Con la
-     mangueta entera (rocker_drop 0.244397) K se queda en 2.56; gastandola toda
-     (0.382097) K baja a 1.78 pero no queda direccion que dibujar.  60 % es el
-     punto en que el poste sigue siendo un poste.  K = 1.00 no se alcanza:
-     haria falta 0.521839 y solo hay 0.382097, porque los brazos no se tocan.
-     QUE NO LIMITA, y parecia que si: el chasis.  Su caja va de y -0.009 a
-     0.241 y las ruedas apoyan en y -0.244 (izquierda) y +0.365 (derecha), o
-     sea 0.23 m por fuera a cada lado.  Ninguna rueda pasa por debajo del
-     chasis en ninguna combinacion de los cuatro pivotes pasivos a +-0.6 rad,
-     asi que bajar el chasis no le acerca ninguna rueda.  Barrido completo en
-     test_bogie_drop.py (seccion 8).
+     mangueta entera K se queda en 2.56; gastandola toda K baja a 1.78 pero no
+     queda direccion que dibujar.  K = 1.00 no se alcanza: haria falta
+     0.521839 y solo hay 0.382097, porque los brazos no se tocan.
+     QUE NO LIMITA, y parecia que si: el chasis.  Ninguna rueda pasa por
+     debajo de el en ninguna combinacion de los cuatro pivotes pasivos a
+     +-0.6 rad, asi que bajarlo no le acerca ninguna rueda.  Barrido completo
+     en test_bogie_drop.py (seccion 8).
      Todo lo que cuelga del chasis sube rocker_drop en el marco de base_link,
-     asi que spawn_z BAJA lo mismo (spawn_z = 1.16 - rocker_drop) y los tres sensores suben
-     rocker_drop en su montaje para conservar su altura sobre la huella: el
-     LiDAR y la camara se quedan donde manda sim_config.yaml y cuelgan de un
-     mastil, y el IMU sigue al CM con imu_rise_per_drop.
+     asi que spawn_z BAJA lo mismo (spawn_z = 1.16 - rocker_drop) y los tres
+     sensores suben rocker_drop en su montaje para conservar su altura sobre
+     la huella.
      ========================================================== -->
 <xacro:arg name="rocker_drop" default="0.299477"/>
@@ -301,45 +201,26 @@
      y el chasis lo tienen- asi que esto NO cambia la fisica: masas, inercias,
      juntas y colisiones se quedan byte a byte donde estaban.
-     POR QUE.  Las mallas son un export de CAD con escala propia
-     (0.001417 0.001164 0.001275) y NO se reescalaron con la huella el
-     2026-09-11, asi que se solapaban en pantalla y el modelo no se podia leer
-     a ojo.  Un tubo dibujado ENTRE dos juntas no puede desincronizarse: se
-     recalcula solo con rocker_drop y con bogie_drop, y de paso se lleva por
-     delante el apaño del montante del bogie, que era un tubo de longitud
-     escrita a mano para tapar ese mismo hueco.
+     POR QUE.  Las mallas son un export de CAD con escala propia y no siguen
+     al reescalado de la huella, asi que se solapaban en pantalla y el modelo
+     no se podia leer a ojo.  Un tubo dibujado ENTRE dos juntas no puede
+     desincronizarse: se recalcula solo con rocker_drop y con bogie_drop.
      La RUEDA se queda con su malla: es el unico eslabon cuya forma se compara
-     entre plataformas y su radio (0.178) esta igualado a mano en las tres.
+     entre plataformas y su radio esta igualado a mano en las tres.
      ========================================================== -->
 <!-- ============ LA MALLA DE LA RUEDA, A LA ESCALA DE SU COLISION ============
-     CORREGIDO EL 2026-09-16.  Las seis ruedas llevaban el visual a
-     "0.002588 0.002126 0.002329", que es la escala del export de CAD y NO la
-     de la rueda que se simula.  Sobre un STL de 86 x 50 x 86 unidades eso
-     dejaba un OVALO de 111.3 x 100.1 mm de semieje y 106.3 de ancho, contra
-     un cilindro de colision de 178 de radio y 114.3 de ancho:
-       * la rueda se veia un 44 % PEQUEÑA, con el borde de arriba a 200 mm
-         del suelo cuando la panza del chasis esta a 338.7, asi que en Gazebo
-         "las ruedas no llegan al chasis" y el vehiculo parece FLOTAR;
-       * y se veia OVALADA, porque la escala era anisotropa (111.3 en x
-         contra 100.1 en z, un 11 % de diferencia).
-     Y LA SIMULACION NO CAMBIA, que era la duda razonable.  La fisica no usa
-     los visuales -masa, inercia, juntas y colisiones siguen byte a byte- y el
-     LiDAR, que SI los usa porque un gpu_ray ve visuales y no colisiones, no
-     alcanza las ruedas: el rayo mas rasante que podria tocar una llanta pide
-     30.5 grados bajo la horizontal con la malla nueva (36.0 con la vieja) y
-     el anillo mas bajo del VLP-16 va a 15.0, ademas de un <range><min> de
-     0.3 m.  O sea que las ruedas no salian en la nube y siguen sin salir; lo
-     unico que cambia es que el dibujo ya coincide con lo que se simula, asi
-     que NO hay que repetir ninguna corrida por esto.  Medido con
-     ve_ruedas.py sobre los seis links.
-     ESCALA NUEVA = (2r/86, ancho/50, 2r/86) = 0.00413953 0.002286 0.00413953
-     Y HAY QUE RECALCULAR EL origin DEL VISUAL, que es el fallo silencioso:
-     en URDF el vertice cae en origin + escala * v, asi que al cambiar la
-     escala la malla se DESPLAZA.  Cada uno de los seis origin se ha sacado
-     para que el centro de la caja envolvente del STL caiga en el centro del
-     cilindro de colision, (0, +-0.052315, 0).  Comprobado sobre el URDF
-     generado: los seis visuales dan 178.00 / 57.15 / 178.00 mm de semieje y
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